File: cccamp23_nametag.kicad_pcb (KiCad board)
At the start: 2 copper layers, 85 x 53 mm, 47 parts, among them Q1 MMBT3904, Q2 MMBT3904, Q3 MMBT3904, SW1 SW_Push_DPDT, SW2 SW_SPST, U1 ATtiny402-SS, U2 ap7375-3.3V

Commit message: final1
Parts:
- removed D10, D11, D12, D13: WS2812B_MINI, nametag_hardware_footprints:ws2812b_mini
- removed D14, D15, D16, D17: WS2812B, nametag_hardware_footprints:ws2812b_micro
- removed X1, X2, X3, X4, X5: ~, nametag_hardware_footprints:repatch
- D1: renamed from D5; value WS2812B -> ws2812b_micro
- D2: renamed from D6; value WS2812B -> ws2812b_micro
- D3: renamed from D1; value WS2812B_MINI -> ws2812b_mini
- D4: renamed from D2; value WS2812B_MINI -> ws2812b_mini
- D5: renamed from D8; value WS2812B -> ws2812b_micro
- D6: renamed from D7; value WS2812B -> ws2812b_micro
- D7: renamed from D4; value WS2812B_MINI -> ws2812b_mini
- D8: renamed from D3; value WS2812B_MINI -> ws2812b_mini
- R1, R5, R6, R8: value tbd -> 10K
- R2, R3: value tbd -> 220R
- R4: value 10K -> 220R
- U1: value ATtiny402-SS -> ap7375-3.3V; footprint Package_SO:SOIC-8_3.9x4.9mm_P1.27mm -> Package_TO_SOT_SMD:SOT-23
- U2: value ap7375-3.3V -> ATtiny402-SS; footprint Package_TO_SOT_SMD:SOT-23 -> Package_SO:SOIC-8_3.9x4.9mm_P1.27mm
- moved TP3 61.9 mm to (64.0, 62.8)
- moved TP1 60.4 mm to (64.0, 57.7)
- moved TP4 59.1 mm to (64.0, 60.2)
- moved SW1 53.2 mm to (142.5, 76.0), turned to -90 degrees
- moved BT1 53.0 mm to (129.0, 91.0)
- moved BT2 53.0 mm to (76.0, 91.0)
- moved SW2 45.4 mm to (138.8, 54.8), turned to 0 degrees
- moved C1 43.7 mm to (137.2, 69.2)
- moved TP2 41.7 mm to (141.2, 69.2)
- moved R1 41.6 mm to (105.8, 72.2), turned to -90 degrees
- moved C2 40.8 mm to (137.2, 75.8), turned to 0 degrees
- moved R2 40.4 mm to (106.8, 80.2)
- moved U1 36.3 mm to (137.2, 72.5), turned to 90 degrees
- moved R3 34.1 mm to (102.5, 80.2)
- moved Q1 26.8 mm to (106.8, 76.2), turned to -90 degrees
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Connections:
- D1 pad 1: +5V -> Net-(D1-DOUT)
- D1 pad 2: Net-(D1-DOUT) -> +5V
- D2 pad 1: +5V -> Net-(D2-DOUT)
- D2 pad 2: Net-(D2-DOUT) -> +5V
- D3 pad 1: Net-(D1-DOUT) -> Net-(D3-DOUT)
- D3 pad 3: /LED_Data -> Net-(D2-DOUT)
- D4 pad 1: Net-(D2-DOUT) -> Net-(D4-DOUT)
- D4 pad 3: Net-(D1-DOUT) -> Net-(D3-DOUT)
- D5 pad 1: +5V -> Net-(D5-DOUT)
- D5 pad 2: unconnected-(D8-DOUT-Pad2) -> +5V
- D5 pad 4: Net-(D3-DOUT) -> Net-(D4-DOUT)
- D6 pad 1: +5V -> Net-(D6-DOUT)
- D6 pad 2: Net-(D3-DOUT) -> +5V
- D6 pad 4: Net-(D2-DOUT) -> Net-(D5-DOUT)
- D7 pad 1: unconnected-(D4-DOUT-Pad1) -> Net-(D7-DOUT)
- D7 pad 3: Net-(D3-DOUT) -> Net-(D6-DOUT)
- D8 pad 1: Net-(D3-DOUT) -> unconnected-(D8-DOUT-Pad1)
- D8 pad 3: Net-(D2-DOUT) -> Net-(D7-DOUT)
- R1 pad 1: /B -> /Control_B
- R1 pad 2: /Col_B -> Net-(Q1-B)
- R2 pad 1: /G -> /B
- R2 pad 2: /Col_G -> /Col_B
- R3 pad 1: /R -> /G
- R3 pad 2: /Col_R -> /Col_G
- R4 pad 1: /Switch -> /R
- R4 pad 2: +5V -> /Col_R
- R5 pad 1: /Control_B -> /Control_G
- R5 pad 2: Net-(Q1-B) -> Net-(Q2-B)
- R6 pad 1: /Control_G -> /Control_R
- R6 pad 2: Net-(Q2-B) -> Net-(Q3-B)
- R7 pad 1: /Control_R -> +5V
- R7 pad 2: Net-(Q3-B) -> Net-(U2-~{RESET}/PA0)
- R8 pad 1: +5V -> /Switch
- R8 pad 2: Net-(U1-~{RESET}/PA0) -> +5V
- TP4 pad 1: Net-(U1-~{RESET}/PA0) -> Net-(U2-~{RESET}/PA0)
- U1 pad 1: +5V -> /SW_VCC
- U1 pad 2: Net-(U1-PA6) -> +5V
- U1 pad 3: Net-(U1-PA7) -> GND
- U2 pad 1: /SW_VCC -> +5V
- U2 pad 2: +5V -> /Switch
- U2 pad 3: GND -> /Control_B
Routing:
- net Net-(D2-DOUT): track 123.7 -> 10.9 mm, vias 3 -> 0
- net Net-(D1-DOUT): track 101.6 -> 7.08 mm
- net Net-(D7-DOUT): track 0.00 -> 78.2 mm
- net Net-(D3-DOUT): track 131.8 -> 77.0 mm
- net +5V: track 317.9 -> 362.9 mm, vias 6 -> 5
- net Net-(D6-DOUT): track 0.00 -> 42.3 mm
- net Net-(U2-~{RESET}/PA0): track 0.00 -> 41.8 mm
- net /LED_Data: track 83.8 -> 42.6 mm, vias 2 -> 1
- net /B: track 11.6 -> 47.3 mm, vias 0 -> 1
- net /Switch: track 16.0 -> 51.2 mm
- net /G: track 9.80 -> 42.5 mm, vias 0 -> 1
- net /R: track 17.0 -> 37.2 mm, vias 2 -> 1
- net /SW_VCC: track 31.3 -> 13.0 mm
- net Net-(U1-~{RESET}/PA0): track 16.8 -> 0.00 mm
- net /Col_B: track 18.6 -> 2.24 mm
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Other:
- board text added: "Brain"
- board text added: "Designed by HazeCore Infos and Documentation: https://hazeco.re/cccamp-nametag"
- board text added: "Hack Area"
- board text added: "Magic Volt Converter"
- board text added: "Mode"
- board text added: "PRGM"
- board text added: "Power"
- board text added: "Real Fast Switches"
- board text removed: "Designed by HazeCore"
- board text removed: "JLCJLCJLCJLC"
- board text removed: "Program / Reset"
- board text removed: "SW_V"
