File: cccamp23_nametag.kicad_sch (KiCad schematic)
At the start: 46 parts, among them Q1 MMBT3904, Q2 MMBT3904, Q3 MMBT3904, SW1 SW_Push_DPDT, SW2 SW_SPST, U1 ATtiny402-SS, U2 ap7375-3.3V

Commit message: final1
Parts:
- removed D1, D10, D11, D12, D13, D2, D3, D4: WS2812B_MINI, nametag_hardware_footprints:ws2812b_mini, symbol tally2:WS2812B_MINI
- removed D14, D15, D16, D17, D5, D6, D7, D8: WS2812B, nametag_hardware_footprints:ws2812b_micro, symbol LED:WS2812B
- removed X1, X2, X3, X4, X5: ~, nametag_hardware_footprints:repatch, symbol nametag_hardware_symbols:repatch
- added D1, D2, D5, D6: ws2812b_micro, nametag_hardware_footprints:ws2812b_micro, symbol nametag_hardware_symbols:ws2812b_micro
- added D3, D4, D7, D8: ws2812b_mini, nametag_hardware_footprints:ws2812b_mini, symbol nametag_hardware_symbols:ws2812b_mini
- R1: renamed from R5; value tbd -> 10K
- R2: renamed from R1; value tbd -> 220R
- R3: renamed from R2; value tbd -> 220R
- R4: renamed from R3; value tbd -> 220R
- R5: renamed from R6; value tbd -> 10K
- R6: renamed from R7; value tbd -> 10K
- renumbered R8 to R7, R4 to R8, U2 to U1, U1 to U2
Connections:
- net +5V: now also D1.2 (VCC), D2.2 (VCC), D3.4 (VCC), D4.4 (VCC), D5.2 (VCC), D6.2 (VCC), D7.4 (VCC), D8.4 (VCC)
- net Control_B: now also U2.3 (PA7)
- net Control_G: now also U2.4 (PA1)
- net Control_R: now also U2.5 (PA2)
- net GND: now also D1.3 (GND), D2.3 (GND), D3.2 (GND), D4.2 (GND), D5.3 (GND), D6.3 (GND), D7.2 (GND), D8.2 (GND)
- net LED_Data: now also U2.7 (PA3), D1.4 (DIN)
- net Switch: now also U2.2 (PA6)
- new net: D5.1 (DOUT), D6.4 (DIN)
- new net: D4.1 (DOUT), D5.4 (DIN)
- new net: D1.1 (DOUT), D2.4 (DIN)
- new net: D7.1 (DOUT), D8.3 (DIN)
- new net: D6.1 (DOUT), D7.3 (DIN)
- new net: D3.1 (DOUT), D4.3 (DIN)
- new net: D2.1 (DOUT), D3.3 (DIN)

Commit message: update schematic
Other:
- note added: "Adressable LEDs"
- note added: "Microcontroller ATtiny402"
- note added: "Power Supply"
- note added: "RGB-Backlight"
- note added: "RGB-Backlight Driver"
- note added: "User Button"
- note removed: "BK-912-TR JS202011JCQN JS202011JAQN https://www.dfrobot.com/product-1717.html"
- title: (none) -> CCCamp23-Nametag
- moved on the sheet: BT1, BT2, C1, C2, C3, D9, R2, R3, R4, R7, R8, SW1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
